Commit message: 🔧modify: ディレクトリ構造の更新

File: src/robots/mobility/urdf/model.urdf (robot description, URDF)
Before this commit: robot ai_car1, 5 links, 4 joints
Links:
- link caster: geometry collision mesh filename=package://camera_based_rl_isaac/src/robots/mobility/urdf/me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 scale=0.1 0.1 0.1; visual mesh filename=package://camera_based_rl_isaac/src/robots/mobility/urdf/me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 scale=0.1 0.1 0.1
- link chassis: geometry collision mesh filename=package://camera_based_rl_isaac/src/robots/mobility/urdf/me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; visual mesh filename=package://camera_based_rl_isaac/src/robots/mobility/urdf/me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
- link left_wheel: geometry collision mesh filename=package://camera_based_rl_isaac/src/robots/mobility/urdf/me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 scale=0.05 0.12 0.12; visual mesh filename=package://camera_based_rl_isaac/src/robots/mobility/urdf/me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 scale=0.05 0.12 0.12
- link right_wheel: geometry collision mesh filename=package://camera_based_rl_isaac/src/robots/mobility/urdf/me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 scale=0.05 0.12 0.12; visual mesh filename=package://camera_based_rl_isaac/src/robots/mobility/urdf/me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 scale=0.05 0.12 0.12
