Commit message: 🐛fix: robot model

File: assets/robots/mobility/urdf/model.urdf (robot description, URDF)
Before this commit: robot mobility, 5 links, 4 joints
Joints:
- removed joint caster_joint
- added joint caster_wheel_joint: type revolute, parent chassis, child caster, origin xyz=-0.8 0 0 rpy=0 0 1.57, axis 1 0 0
- joint left_wheel_joint: origin xyz=0 -0.3 0 rpy=0 0 0 -> xyz=0 0.3 0 rpy=0 0 0
- joint right_wheel_joint: origin xyz=0 0.3 0 rpy=0 0 0 -> xyz=0 -0.3 0 rpy=0 0 0

Commit message: ✨feat: caster yaw link model

File: assets/robots/mobility/urdf/model.urdf (robot description, URDF)
Before this commit: robot mobility, 5 links, 4 joints
Links:
- added link caster_roll_link
- added link caster_yaw_link
Joints:
- removed joint caster_wheel_joint
- added joint caster_mount_joint: type fixed, parent caster_roll_link, child caster, origin xyz=0 0 0 rpy=0 0 0
- added joint caster_roll_joint: type revolute, parent caster_yaw_link, child caster_roll_link, origin xyz=0 0 0 rpy=0 0 0, axis 1 0 0
- added joint caster_yaw_joint: type revolute, parent chassis, child caster_yaw_link, origin xyz=-0.8 0 -0.02 rpy=0 0 1.57, axis 0 0 1, limit lower=-0.5236 upper=0.5236

Commit message: ✨feat: ロボットモデルの改善

File: assets/robots/mobility/urdf/model.urdf (robot description, URDF)
Before this commit: robot mobility, 7 links, 6 joints
Links:
- link left_wheel: geometry collision mesh filename=package://camera_based_rl_isaac/src/robots/mobility/urdf/me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 scale=0.1 0.12 0.12; visual mesh filename=package://camera_based_rl_isaac/src/robots/mobility/urdf/me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 scale=0.1 0.12 0.12
- link right_wheel: geometry collision mesh filename=package://camera_based_rl_isaac/src/robots/mobility/urdf/me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 scale=0.1 0.12 0.12; visual mesh filename=package://camera_based_rl_isaac/src/robots/mobility/urdf/me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 scale=0.1 0.12 0.12

Commit message: ✨feat: mass

File: assets/robots/mobility/urdf/model.urdf (robot description, URDF)
Before this commit: robot mobility, 7 links, 6 joints
Links:
- link caster: mass 10.0 -> 16.0
- link left_wheel: mass 7.0 -> 12.0
- link right_wheel: mass 7.0 -> 12.0
